File: Core-ESP32.sch (EAGLE design)
At the start: 58 parts, among them J2 CONNECTOR-GROVE-4P-2.0-347013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, Q1 BSS138, Q10 BSS138, Q11 BSS138, Q12 BSS138, Q13 BSS138, Q2 BSS138, Q3 BSS138, Q4 BSS138, Q5 BSS138, Q6 BSS138, Q7 BSS138, Q8 BSS138, Q9 BSS138

Commit message: 2.0
Parts:
- removed C4: 10uF, SPCoast:CAP0805
- removed ESP32: ESP32, SPCoast:ESP32
- removed JP3: (no value), SparkFun-Connectors:M06LOCK
- added I2CLED32, I2CLED64: (no value), SPCoast:CONNECTOR-M04LOCK
- added IO-A, IO-B, IO-C: (no value), SparkFun-Connectors:M06LOCK
- added J5: (no value), SPCoast:CONNECTOR-RJ25-43860-2-MOLEX
- added R27: 10k, SPCoast:R0805-RES
- added U$1: ESP32-GEEKCREITDOITV1, SPCoast:ESP32-GEEKCREITDOITV1
- C2: value 150uF -> 1.0uF; device SPCoast:CAP-POL0810 -> SPCoast:CAP0805
- C3: value 1.0uF -> 10uF
- J1: device SPCoast:CONNECTOR-DC-POWER-RA -> SPCoast:CONNECTOR-RJ25-43860-2-MOLEX
- J2: value CONNECTOR-GROVE-4P-2.0-3470130P1 -> (none); device SPCoast:CONNECTOR-GROVE-4P-2.0-3470130P1 -> SPCoast:CONNECTOR-DC-POWER-RA
- J3: value (none) -> CONNECTOR-GROVE-4P-2.0-3470130P1; device SPCoast:CONNECTOR-RJ25-43860-2-MOLEX -> SPCoast:CONNECTOR-GROVE-4P-2.0-3470130P1
- JP1: value 5v I2C Power -> LED
- JP2: value (none) -> 5v I2C Power; device SparkFun-Connectors:M06LOCK -> SparkFun-Connectors:M02LOCK
- R1: value 10k -> 220R
- VR5.0: value 5v -> 78M05B
- renumbered LED1 to MATRIX1, LED2 to MATRIX2
Connections:
- removed net D15H: J3.3, JP2.3, Q4.D, R17.1
- removed net D26H: J4.5, JP3.5, Q10.D, R23.1
- removed net D36: ESP32.GPIO36, Q8.S, R10.1
- removed net D36H: J4.3, JP3.3, Q8.D, R21.1
- removed net RXH: J3.4, JP2.4, Q5.D, R18.1
- removed net TXH: J3.5, JP2.5, Q6.D, R19.1
- new net D18: Q6.S, R6.1, U$1.GPIO18
- new net D18H: IO-C.2, J5.2, Q6.D, R19.1
- new net D19: Q7.S, R7.1, U$1.GPIO19
- new net D19H: IO-C.3, J5.3, Q7.D, R20.1
- new net D23: Q10.S, R10.1, U$1.GPIO23
- new net D23H: IO-C.4, J5.4, Q10.D, R23.1
- new net D27: U$1.GPIO27
- new net D32: U$1.GPIO32
- new net D33: U$1.GPIO33
- new net D4: Q4.S, R4.1, U$1.GPIO4
- new net D4H: IO-B.4, J4.4, Q4.D, R17.1
- new net D5: Q5.S, R5.1, U$1.GPIO5
- new net D5H: IO-B.5, J4.5, Q5.D, R18.1
- new net N$1: JP1.1, R1.1
- new net RX2: IO-A.5, J1.5, U$1.RX2
- new net TX2: IO-A.4, J1.4, U$1.TX2
- net +3V3: now also I2CLED32.3, I2CLED64.3, IO-A.1, J1.1, R2.2, R4.2, U$1.+3V3; no longer ESP32.+3V3, R15.2
- net +9V: now also C2.1, J2.1, J3.3, J3.4; no longer C2.+, C3.1, J1.1, J2.3, J2.4
- net D0: now also Q2.S, R2.1, U$1.GPIO0; no longer ESP32.GPIO0, Q3.S, R5.1
- net D0H: now also IO-B.2, J4.2, Q2.D, R15.1; no longer J3.2, JP2.2, Q3.D, R16.1
- net D12: now also Q13.S, R13.1, U$1.GPIO12; no longer ESP32.GPIO12, Q12.S, R14.1
- net D12H: now also Q13.D, R26.1; no longer Q12.D, R25.1
- net D13: now also Q1.S, R14.1, U$1.GPIO13; no longer ESP32.GPIO13, Q13.S, R15.1
- net D13H: now also Q1.D, R27.1; no longer Q13.D, R26.1
- net D14: now also Q12.S, R12.1, U$1.GPIO14; no longer ESP32.GPIO14, Q11.S, R13.1
- net D14H: now also Q12.D, R25.1; no longer Q11.D, R24.1
- net D15: now also JP1.2, U$1.GPIO15; no longer ESP32.GPIO15, Q4.S, R6.1
- net D2: now also Q3.S, R3.1, U$1.GPIO2; no longer ESP32.GPIO2, Q7.S, R9.1
- net D25: now also Q11.S, U$1.GPIO25; no longer ESP32.GPIO25, Q9.S
- net D25H: now also IO-C.5, J5.5, Q11.D, R24.1; no longer J4.4, JP3.4, Q9.D, R22.1
- net D26: now also U$1.GPIO26; no longer ESP32.GPIO26, Q10.S, R12.1
- net D2H: now also IO-B.3, J4.3, Q3.D, R16.1; no longer J4.2, JP3.2, Q7.D, R20.1
- net GND: now also C2.2, I2CLED32.4, I2CLED64.4, IO-A.6, IO-B.6, IO-C.6, J1.6, J2.3, J3.1, J3.2, J5.6, U$1.GND; no longer C2.-, C4.2, ESP32.GND, J1.2, J1.3, J2.1, J3.6, JP2.6, JP3.6
- net N$44: now also JP2.1; no longer JP1.1
- net RX: now also IO-A.3, J1.3, U$1.RX1; no longer ESP32.RX, Q5.S, R7.1
- net SCL: now also I2CLED32.2, I2CLED64.2, Q9.S, R9.1, U$1.SCL; no longer ESP32.SCL, Q2.S, R3.1
- net SCLH: now also Q9.D, R22.1; no longer Q2.D, R4.1
- net SDA: now also I2CLED32.1, I2CLED64.1, Q8.S, R8.1, U$1.SDA; no longer ESP32.SDA, Q1.S, R1.1
- net SDAH: now also Q8.D, R21.1; no longer Q1.D, R2.1
- net TX: now also IO-A.2, J1.2, U$1.TX1; no longer ESP32.TX, Q6.S, R8.1
- net VCCIO: now also C3.1, IO-B.1, IO-C.1, J5.1, JP2.2, R15.2, R27.2, U$1.+5V; no longer C4.1, ESP32.+5V, J3.1, JP1.2, JP2.1, JP3.1, R2.2, R4.2
Other:
- note added: "A"
- note added: "ESP32 I/O Level Shifters"
- note added: "Geekcreit/DOIT ESP32"
- note added: "IO & I2C Adapter for Geekcreit ESP32"
- note added: "IO-B"
- note added: "IO-C"
- note added: "LED Matrix"
- note added: "Processor carrier board for Geekcreit ESP32 Breaks out 5v I2C, IO4 style headers and Matrix Display"
- note removed: "IO & I2C Adapter for WeMOS Lolin ESP32 + OLED"
- note removed: "Problem: board does not boot with GPIO 12 pulled high"
- note removed: "Processor carrier board for WeMOS Lolin ESP32 with OLED Breaks out 5v I2C, IO4 style header for direct IO, Maintainer Call and Matrix Display"
- note removed: "WeMos / Lolin ESP32-OLED"

Commit message: 2.1
Parts:
- removed JP1: LED, SparkFun-Connectors:M02LOCK
- removed JP2: 5v I2C Power, SparkFun-Connectors:M02LOCK
- removed MATRIX1, MATRIX2: LEDMATRIX, SPCoast:LEDMATRIX
- removed R1: 220R, SPCoast:R0805-RES
- added I2CLED1: (no value), SPCoast:CONNECTOR-M04LOCK
- added J6: (no value), SPCoast:CONNECTOR-RJ25-43860-2-MOLEX
- added Q14: BSS138, SPCoast:MOSFET-N-BSS138-SOT23
- added R28, R29: 10k, SPCoast:R0805-RES
- BOARD: device SPCoast:BOARD80X150 -> SPCoast:BOARD80X100-NOHOLES
Connections:
- removed net D0H: IO-B.2, J4.2, Q2.D, R15.1
- removed net D12H: MATRIX2.CS@1, Q13.D, R26.1
- removed net D2H: IO-B.3, J4.3, Q3.D, R16.1
- removed net N$1: JP1.1, R1.1
- removed net N$10: MATRIX1.CLK@1, MATRIX2.CLK@2
- removed net N$3: MATRIX1.DIN, MATRIX2.DOUT
- removed net N$44: I2C.V+, JP2.1
- removed net N$9: MATRIX1.CS@1, MATRIX2.CS@2
- new net D26H: J6.2, Q14.D, R29.1
- new net D27H: J6.4, Q13.D, R26.1
- new net D32H: IO-B.4, J4.4, Q2.D, R15.1
- new net D33H: IO-B.5, J4.5, Q3.D, R16.1
- net +3V3: now also I2CLED1.3, Q14.G, R28.2; no longer R1.2
- net D0: no longer Q2.S, R2.1
- net D12: no longer Q13.S, R13.1
- net D13H: now also J6.5; no longer MATRIX2.CLK@1
- net D14H: now also J6.3; no longer MATRIX2.DIN
- net D15: no longer JP1.2
- net D2: no longer Q3.S, R3.1
- net D26: now also Q14.S, R28.1
- net D27: now also Q13.S, R13.1
- net D32: now also Q2.S, R2.1
- net D33: now also Q3.S, R3.1
- net D4H: now also IO-B.2, J4.2; no longer IO-B.4, J4.4
- net D5H: now also IO-B.3, J4.3; no longer IO-B.5, J4.5
- net GND: now also I2CLED1.4, J6.6; no longer MATRIX1.G@1, MATRIX1.G@2, MATRIX2.G@1, MATRIX2.G@2
- net SCL: now also I2CLED1.2
- net SDA: now also I2CLED1.1
- net VCCIO: now also I2C.V+, J6.1, R29.2; no longer JP2.2, MATRIX1.V+@1, MATRIX1.V+@2, MATRIX2.V+@1, MATRIX2.V+@2
Other:
- note added: "2.1"
- note added: "LED"
- note removed: "CS"
- note removed: "DATA"
- note removed: "clock"
- moved on the sheet: I2CLED32, I2CLED64, IO-A, IO-B, IO-C, J1, J4, J5, Q10, Q11, Q2, Q3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

Commit message: 2.2
Parts:
- C2, C3: device SPCoast:CAP0805 -> SPCoast:CAP0603
- R10, R11, R12, R13, R14, R15, R16, R17, R18, R19, R2, R20, R21, R22, R23, R24, R25, R26, R27, R28, R29, R3, R4, R5, R6, R7, R8, R9: device SPCoast:R0805-RES -> SPCoast:R0603-RES
Other:
- note added: "2.2"
- note added: "Processor carrier board for Geekcreit ESP32 Breaks out 5v I2C, IO4 style headers and Matrix Display 2.1->2.2: change from 0805 to 0603 footprints"
- note removed: "2.1"
- note removed: "Processor carrier board for Geekcreit ESP32 Breaks out 5v I2C, IO4 style headers and Matrix Display"

Commit message: 2.3
Parts:
- added MT1, MT2, MT3, MT4: MOUNTINGHOLE, SPCoast:MOUNTINGHOLE
Other:
- note added: "2.3"
- note removed: "2.2"
Changed lines of the file:
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@@
 <grid distance="0.1" unitdist="inch" unit="inch" style="lines" multiple="1" display="no" altdistance="0.01" altunitdist="inch" altunit="inch"/>
 <layers>
-<layer number="1" name="Top" color="4" fill="1" visible="yes" active="no"/>
-<layer number="2" name="Route2" color="1" fill="3" visible="yes" active="no"/>
-<layer number="3" name="Route3" color="4" fill="3" visible="yes" active="no"/>
-<layer number="4" name="Route4" color="1" fill="4" visible="yes" active="no"/>
-<layer number="5" name="Route5" color="4" fill="4" visible="yes" active="no"/>
-<layer number="6" name="Route6" color="1" fill="8" visible="yes" active="no"/>
-<layer number="7" name="Route7" color="4" fill="8" visible="yes" active="no"/>
-<layer number="8" name="Route8" color="1" fill="2" visible="yes" active="no"/>
-<layer number="9" name="Route9" color="4" fill="2" visible="yes" active="no"/>
-<layer number="10" name="Route10" color="1" fill="7" visible="yes" active="no"/>
-<layer number="11" name="Route11" color="4" fill="7" visible="yes" active="no"/>
-<layer number="12" name="Route12" color="1" fill="5" visible="yes" active="no"/>
-<layer number="13" name="Route13" color="4" fill="5" visible="yes" active="no"/>
-<layer number="14" name="Route14" color="1" fill="6" visible="yes" active="no"/>
-<layer number="15" name="Route15" color="4" fill="6" visible="yes" active="no"/>
-<layer number="16" name="Bottom" color="2" fill="1" visible="yes" active="no"/>
-<layer number="17" name="Pads" color="2" fill="1" visible="yes" active="no"/>
-<layer number="18" name="Vias" color="3" fill="1" visible="yes" active="no"/>
-<layer number="19" name="Unrouted" color="6" fill="1" visible="yes" active="no"/>
-<layer number="20" name="Dimension" color="15" fill="1" visible="yes" active="no"/>
-<layer number="21" name="tPlace" color="27" fill="1" visible="yes" active="no"/>
-<layer number="22" name="bPlace" color="17" fill="1" visible="yes" active="no"/>
-<layer number="23" name="tOrigins" color="30" fill="1" visible="yes" active="no"/>
-<layer number="24" name="bOrigins" color="15" fill="1" visible="yes" active="no"/>
-<layer number="25" name="tNames" color="7" fill="1" visible="yes" active="no"/>
-<layer number="26" name="bNames" color="34" fill="1" visible="yes" active="no"/>
-<layer number="27" name="tValues" color="22" fill="1" visible="yes" active="no"/>
-<layer number="28" name="bValues" color="7" fill="1" visible="yes" active="no"/>
+<layer number="1" name="Top" color="4" fill="1" visible="no" active="no"/>
+<layer number="2" name="Route2" color="1" fill="3" visible="no" active="no"/>
+<layer number="3" name="Route3" color="4" fill="3" visible="no" active="no"/>
+<layer number="4" name="Route4" color="1" fill="4" visible="no" active="no"/>
+<layer number="5" name="Route5" color="4" fill="4" visible="no" active="no"/>
+<layer number="6" name="Route6" color="1" fill="8" visible="no" active="no"/>
+<layer number="7" name="Route7" color="4" fill="8" visible="no" active="no"/>
+<layer number="8" name="Route8" color="1" fill="2" visible="no" active="no"/>
+<layer number="9" name="Route9" color="4" fill="2" visible="no" active="no"/>
+<layer number="10" name="Route10" color="1" fill="7" visible="no" active="no"/>
+<layer number="11" name="Route11" color="4" fill="7" visible="no" active="no"/>
+<layer number="12" name="Route12" color="1" fill="5" visible="no" active="no"/>
+<layer number="13" name="Route13" color="4" fill="5" visible="no" active="no"/>
+<layer number="14" name="Route14" color="1" fill="6" visible="no" active="no"/>
+<layer number="15" name="Route15" color="4" fill="6" visible="no" active="no"/>
+<layer number="16" name="Bottom" color="2" fill="1" visible="no" active="no"/>
+<layer number="17" name="Pads" color="2" fill="1" visible="no" active="no"/>
+<layer number="18" name="Vias" color="3" fill="1" visible="no" active="no"/>
+<layer number="19" name="Unrouted" color="6" fill="1" visible="no" active="no"/>
+<layer number="20" name="Dimension" color="15" fill="1" visible="no" active="no"/>
+<layer number="21" name="tPlace" color="27" fill="1" visible="no" active="no"/>
+<layer number="22" name="bPlace" color="17" fill="1" visible="no" active="no"/>
+<layer number="23" name="tOrigins" color="30" fill="1" visible="no" active="no"/>
+<layer number="24" name="bOrigins" color="15" fill="1" visible="no" active="no"/>
+<layer number="25" name="tNames" color="7" fill="1" visible="no" active="no"/>
+<layer number="26" name="bNames" color="34" fill="1" visible="no" active="no"/>
+<layer number="27" name="tValues" color="22" fill="1" visible="no" active="no"/>
+<layer number="28" name="bValues" color="7" fill="1" visible="no" active="no"/>
 <layer number="29" name="tStop" color="5" fill="1" visible="no" active="no"/>
 <layer number="30" name="bStop" color="7" fill="6" visible="no" active="no"/>
@@
 <layer number="35" name="tGlue" color="7" fill="4" visible="no" active="no"/>
 <layer number="36" name="bGlue" color="7" fill="5" visible="no" active="no"/>
-<layer number="37" name="tTest" color="7" fill="1" visible="yes" active="no"/>
-<layer number="38" name="bTest" color="7" fill="1" visible="yes" active="no"/>
+<layer number="37" name="tTest" color="7" fill="1" visible="no" active="no"/>
+<layer number="38" name="bTest" color="7" fill="1" visible="no" active="no"/>
 <layer number="39" name="tKeepout" color="4" fill="11" visible="no" active="no"/>
 <layer number="40" name="bKeepout" color="3" fill="11" visible="no" active="no"/>
@@
 <layer number="44" name="Drills" color="2" fill="1" visible="no" active="no"/>
 <layer number="45" name="Holes" color="35" fill="1" visible="no" active="no"/>
-<layer number="46" name="Milling" color="1" fill="1" visible="yes" active="no"/>
-<layer number="47" name="Measures" color="21" fill="1" visible="yes" active="no"/>
-<layer number="48" name="Document" color="24" fill="1" visible="yes" active="no"/>
-<layer number="49" name="Reference" color="7" fill="1" visible="yes" active="no"/>
-<layer number="50" name="dxf" color="7" fill="1" visible="yes" active="no"/>
-<layer number="51" name="tDocu" color="22" fill="1" visible="yes" active="no"/>
-<layer number="52" name="bDocu" color="7" fill="1" visible="yes" active="no"/>
-<layer number="53" name="tGND_GNDA" color="7" fill="9" visible="yes" active="no"/>
-<layer number="54" name="bGND_GNDA" color="1" fill="9" visible="yes" active="no"/>
-<layer number="56" name="wert" color="7" fill="1" visible="yes" active="no"/>
-<layer number="57" name="tCAD" color="7" fill="1" visible="yes" active="no"/>
-<layer number="59" name="tCarbon" color="7" fill="1" visible="yes" active="no"/>
-<layer number="60" name="bCarbon" color="7" fill="1" visible="yes" active="no"/>
+<layer number="46" name="Milling" color="1" fill="1" visible="no" active="no"/>
+<layer number="47" name="Measures" color="21" fill="1" visible="no" active="no"/>
+<layer number="48" name="Document" color="24" fill="1" visible="no" active="no"/>
+<layer number="49" name="Reference" color="7" fill="1" visible="no" active="no"/>
+<layer number="50" name="dxf" color="7" fill="1" visible="no" active="no"/>
+<layer number="51" name="tDocu" color="22" fill="1" visible="no" active="no"/>
+<layer number="52" name="bDocu" color="7" fill="1" visible="no" active="no"/>
+<layer number="53" name="tGND_GNDA" color="7" fill="9" visible="no" active="no"/>
+<layer number="54" name="bGND_GNDA" color="1" fill="9" visible="no" active="no"/>
+<layer number="56" name="wert" color="7" fill="1" visible="no" active="no"/>
+<layer number="57" name="tCAD" color="7" fill="1" visible="no" active="no"/>
+<layer number="59" name="tCarbon" color="7" fill="1" visible="no" active="no"/>
+<layer number="60" name="bCarbon" color="7" fill="1" visible="no" active="no"/>
 <layer number="90" name="Modules" color="5" fill="1" visible="no" active="no"/>
 <layer number="91" name="Nets" color="2" fill="1" visible="yes" active="yes"/>
@@
 <part name="VCC4" library="supply1" deviceset="VCCIO" device=""/>
 <part name="VCC2" library="supply1" deviceset="VCCIO" device=""/>
+<part name="MT1" library="SPCoast" deviceset="MOUNTINGHOLE" device=""/>
+<part name="MT2" library="SPCoast" deviceset="MOUNTINGHOLE" device=""/>
+<part name="MT3" library="SPCoast" deviceset="MOUNTINGHOLE" device=""/>
+<part name="MT4" library="SPCoast" deviceset="MOUNTINGHOLE" device=""/>
 </parts>
 <sheets>
@@
 Geekcreit ESP32</text>
 <text x="152.908" y="6.35" size="3.81" layer="97">John Plocher</text>
-<text x="235.458" y="6.604" size="3.81" layer="97">2.2</text>
+<text x="235.458" y="6.604" size="3.81" layer="97">2.3</text>
 <text x="149.86" y="38.1" size="1.6764" layer="102">Processor carrier board for Geekcreit ESP32
 Breaks out 5v I2C, IO4 style headers and Matrix Display
@@
 <instance part="V3" gate="GND" x="25.4" y="137.16"/>
 <instance part="VCC2" gate="G$1" x="177.8" y="73.66"/>
+<instance part="MT1" gate="MT1" x="238.76" y="53.34"/>
+<instance part="MT2" gate="MT1" x="238.76" y="68.58"/>
+<instance part="MT3" gate="MT1" x="238.76" y="83.82"/>
+<instance part="MT4" gate="MT1" x="238.76" y="99.06"/>
 </instances>
 <busses>

Commit message: 2.4
Parts:
- added IO-D: (no value), SparkFun-Connectors:M06LOCK
Connections:
- net D13H: now also IO-D.5
- net D14H: now also IO-D.3
- net D26H: now also IO-D.2
- net D27H: now also IO-D.4
- net GND: now also IO-D.6
- net VCCIO: now also IO-D.1
Other:
- note added: "2.4"
- note added: "Processor carrier board for Geekcreit ESP32 Breaks out 5v I2C, IO4 style headers and Matrix Display 2.1->2.2: change from 0805 to 0603 footprints 2.4: codeline is now I2C, add more I/Os"
- note removed: "2.3"
- note removed: "Processor carrier board for Geekcreit ESP32 Breaks out 5v I2C, IO4 style headers and Matrix Display 2.1->2.2: change from 0805 to 0603 footprints"
Changed lines of the file:
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@@
 <setting verticaltext="up"/>
 </settings>
-<grid distance="0.1" unitdist="inch" unit="inch" style="lines" multiple="1" display="no" altdistance="0.01" altunitdist="inch" altunit="inch"/>
+<grid distance="100" unitdist="mil" unit="mil" style="dots" multiple="1" display="yes" altdistance="50" altunitdist="mil" altunit="mil"/>
 <layers>
 <layer number="1" name="Top" color="4" fill="1" visible="no" active="no"/>
@@
 <part name="MT3" library="SPCoast" deviceset="MOUNTINGHOLE" device=""/>
 <part name="MT4" library="SPCoast" deviceset="MOUNTINGHOLE" device=""/>
+<part name="IO-D" library="SparkFun-Connectors" deviceset="M06" device="LOCK"/>
 </parts>
 <sheets>
@@
 Geekcreit ESP32</text>
 <text x="152.908" y="6.35" size="3.81" layer="97">John Plocher</text>
-<text x="235.458" y="6.604" size="3.81" layer="97">2.3</text>
+<text x="235.458" y="6.604" size="3.81" layer="97">2.4</text>
 <text x="149.86" y="38.1" size="1.6764" layer="102">Processor carrier board for Geekcreit ESP32
 Breaks out 5v I2C, IO4 style headers and Matrix Display
-2.1-&gt;2.2: change from 0805 to 0603 footprints</text>
+2.1-&gt;2.2: change from 0805 to 0603 footprints
+2.4: codeline is now I2C, add more I/Os</text>
 <text x="190.5" y="86.36" size="5.08" layer="97">I2C</text>
 <text x="86.36" y="165.1" size="5.08" layer="97">Geekcreit/DOIT
@@
 <instance part="MT3" gate="MT1" x="238.76" y="83.82"/>
 <instance part="MT4" gate="MT1" x="238.76" y="99.06"/>
+<instance part="IO-D" gate="G$1" x="30.48" y="147.32" rot="R180"/>
 </instances>
 <busses>
@@
 <wire x1="40.64" y1="139.7" x2="25.4" y2="139.7" width="0.1524" layer="91"/>
 <pinref part="V3" gate="GND" pin="GND"/>
+<pinref part="IO-D" gate="G$1" pin="6"/>
+<junction x="25.4" y="139.7"/>
 </segment>
 </net>
@@
 <wire x1="40.64" y1="152.4" x2="25.4" y2="152.4" width="0.1524" layer="91"/>
 <pinref part="VCC1" gate="G$1" pin="VCCIO"/>
+<pinref part="IO-D" gate="G$1" pin="1"/>
+<junction x="25.4" y="152.4"/>
 </segment>
 <segment>
@@
 <wire x1="25.4" y1="147.32" x2="22.86" y2="147.32" width="0.1524" layer="91"/>
 <label x="22.86" y="147.32" size="1.016" layer="95" rot="R180" xref="yes"/>
+<pinref part="IO-D" gate="G$1" pin="3"/>
+<junction x="25.4" y="147.32"/>
 </segment>
 </net>
@@
 <wire x1="25.4" y1="144.78" x2="22.86" y2="144.78" width="0.1524" layer="91"/>
 <label x="22.86" y="144.78" size="1.016" layer="95" rot="R180" xref="yes"/>
+<pinref part="IO-D" gate="G$1" pin="4"/>
+<junction x="25.4" y="144.78"/>
 </segment>
 </net>
@@
 <wire x1="25.4" y1="142.24" x2="22.86" y2="142.24" width="0.1524" layer="91"/>
 <label x="22.86" y="142.24" size="1.016" layer="95" rot="R180" xref="yes"/>
+<pinref part="IO-D" gate="G$1" pin="5"/>
+<junction x="25.4" y="142.24"/>
 </segment>
 </net>
@@
 <wire x1="25.4" y1="149.86" x2="22.86" y2="149.86" width="0.1524" layer="91"/>
 <label x="22.86" y="149.86" size="1.016" layer="95" rot="R180" xref="yes"/>
-</segment>
-</net>
+<pinref part="IO-D" gate="G$1" pin="2"/>
+<junction x="25.4" y="149.86"/>
+</segment>
+</net>
